File: hardware/Badge_Tropicon_2026.kicad_sch (KiCad schematic)
At the start: 24 parts, among them U2 Si4463, Y1 30MHz

Commit message: feat(Hw):Update_Schematic
Parts:
- removed AE1: Antenna, symbol Device:Antenna
- removed C1: 1uF, symbol Device:C_Small
- removed C2: 100nF, symbol Device:C_Small
- removed C3: 3.3pF, symbol Device:C
- removed L3: 11nH, symbol Device:L
- removed L4: 10nH, symbol Device:L
- added AE1, AE2: Antenna_Shield, symbol Device:Antenna_Shield
- added C1: 100nF, symbol Device:C
- added C13, C14, C15, C3: 10uF, Capacitor_SMD:C_0603_1608Metric, symbol Device:C_Small
- added C16, C17, C18, C19, C20, C21: 0.1uF, Capacitor_SMD:C_0603_1608Metric, symbol Device:C_Small
- added C2: 1uF, symbol Device:C
- added C3: 1uF, Capacitor_SMD:C_0603_1608Metric, symbol Device:C_Small
- added D1: MBR120, Diode_SMD:D_SOD-123F, symbol Diode:MBR340
- added F1: 0.75A, Fuse:Fuse_0603_1608Metric, symbol Device:Fuse_Small
- added J1: Battery, Footprints:BAT-TH_BH-AAA-A1AJ024, symbol Connector:Screw_Terminal_01x02
- added P1: USB_C_Plug_USB2.0, Footprints:C393939, symbol HunterCat-NFC-rescue:USB_C_Plug_USB2.0-Connector
- added Q1: DMG3415U-7, Package_TO_SOT_SMD:SOT-23, symbol Device:Q_PMOS_GSD
- added R5: 3.3K, Resistor_SMD:R_0603_1608Metric, symbol Device:R_Small
- added R6: 100K, Resistor_SMD:R_0603_1608Metric, symbol Device:R_Small
- added R7: 10K, Resistor_SMD:R_0603_1608Metric, symbol Device:R_Small
- added R8, R9: 5k1, Resistor_SMD:R_0603_1608Metric, symbol Device:R_Small
- added SW1: ON, Footprints:MSK12C02, symbol Switch:SW_SPST
- added SW2, SW3, SW4, SW5, SW6, SW7: ~, Button_Switch_SMD:SW_SPST_TL3342, symbol Switch:SW_Push
- added U1: VGdd79S915N0S1, symbol Library:VGdd79S915N0S1
- added U3: AHT30, symbol Library:AHT30
- added U4: ESP32-C6-WROOM-1U-N4, Footprints:ESP32C6WROOM1N4, symbol Minino:ESP32-C6-WROOM-1U-N8
- added U5: XC6220B331MR-G, Package_TO_SOT_SMD:SOT-23-5, symbol HunterCat-NFC-rescue:AP2112K-3.3-Regulator_Linear
- C4: value 3.3pF -> 220pF
- C5: value 4.7pF -> 12pF
- C6: value 1.11pF -> 6pF
- L1: value 100nH -> 240nH
- L2: value 13nH -> 160nH
Connections:
- net +3V3 is gone; now on net +3.3V: R1.1, U2.6 (VDD), U2.8 (VDD)
- net CLK: now also U1.4 (SCK)
- net CS: now also U1.5 (NSS)
- net GND: now also C10.2, C11.2, C12.2, C5.1, C7.2, C8.2, C9.2, AE1.2 (Shield), AE2.2 (Shield), C1.2, C13.2, C14.2, C15.2, C16.1, C17.1, C18.1, C19.1, C2.2, C20.1, C21.1, C3.2, C3.2, J1.1 (Pin_1), P1.A1 (GND), P1.A12 (GND), P1.B1 (GND), P1.B12 (GND), P1.S1 (SHIELD), R6.2, R8.1, R9.1, SW2.1, SW3.1, SW4.1, SW5.1, SW6.1, SW7.1, U1.12 (GND), U1.13 (GND), U1.7 (GND), U1.9 (GND), U3.5 (GND), U4.1 (GND), U4.28 (GND), U4.29 (GND), U4.30 (GND), U4.31 (GND), U4.32 (GND), U4.33 (GND), U4.34 (GND), U4.35 (GND), U4.36 (GND), U4.37 (GND), U5.2 (GND)
- net SDI: now also U1.2 (MISO)
- net SDO: now also U1.3 (MOSI)
- net +3.3V: now reaches C11.1
- net +3.3V: now also C12.1, C7.1, R2.1, R3.1, R4.1, C1.1, C13.1, C15.1, C2.1, C3.1, C3.1, R5.2, R7.2, U1.6 (VCC), U4.2 (3V3), U5.5 (VOUT)
- net Rxp: now reaches L1.1
- net Rxp: now also C5.2, L2.1, U2.2 (RXp)
- net Rxn: now reaches L1.2
- net Rxn: now also C6.1, U2.3 (RXn)
- net at L2.2: now also C4.1, C6.2
- net at C4.2: now also AE1.1 (A)
- net at L5.1: now also C9.1, U1.14 (ANT)
- net at L5.2: now also C10.1, AE2.1 (A)
- net at R3.2: now also C8.1, U3.2 (VDD)
- net SCL: now reaches R2.2
- net SCL: now also U3.3 (SCL), U4.7 (IO7)
- net SDA: now reaches R4.2
- net SDA: now also U3.4 (SDA), U4.6 (IO6)
- new net: D1.1 (K), Q1.2 (S), SW1.2 (B)
- new net: C14.1, SW1.3 (A), U5.1 (VIN), U5.3 (EN)
- new net: F1.1, P1.A4 (VBUS), P1.A9 (VBUS), P1.B4 (VBUS), P1.B9 (VBUS)
- new net: R5.1, U4.10 (IO8)
- new net: P1.A5 (CC), R8.2
- new net: P1.B5 (VCONN), R9.2
- new net +BATT: J1.2 (Pin_2), Q1.3 (D)
- new net BOOT: C16.2, SW2.2, U4.16 (IO18)
- new net D+: P1.A6 (D+), U4.14 (IO13)
- new net D-: P1.A7 (D-), U4.13 (IO12)
- new net DOWN: C20.2, SW7.2
- new net EN: C17.2, R7.1, SW3.2, U4.3 (EN)
- new net LEFT: C18.2, SW5.2
- new net RIGHT: C19.2, SW6.2
- new net UP: C21.2, SW4.2
- new net VBUS: D1.2 (A), F1.2, Q1.1 (G), R6.1
- no-connect marks 0 -> 5
Other:
- note added: "AHT30"
- note added: "BUTTONS"
- note added: "ESP32-C6"
- note added: "REGULATOR"
- note added: "SI4463"
- note added: "USB-C"
- note added: "VGdd79S915N0S1"
- moved on the sheet: C10, C11, C12, C4, C5, C6, C7, C8, C9, L1, L2, L5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

Commit message: feat(Hw):Update_Schematic
Parts:
- C10, C9: value C -> 6.8pF
- L5: value L -> 10nH
Connections:
- net DOWN: now also U4.23 (IO15)
- net IO0: now also U4.18 (IO20)
- net IO1: now also U4.19 (IO21)
- net IO2: now also U4.20 (IO22)
- net IO3: now also U4.21 (IO23)
- net IRQ: now also U4.17 (IO19)
- net LEFT: now also U4.12 (IO11)
- net RIGHT: now also U4.15 (IO9)
- net SCL: now also U4.9 (IO1); no longer U4.7 (IO7)
- net SDA: now also U4.8 (IO0); no longer U4.6 (IO6)
- net UP: now also U4.26 (IO3)
- net RST: now reaches U1.1 (RST)
- net RST: now also U4.4 (IO4)
- net DIO: now reaches U1.10 (DIO1)
- net DIO: now also U4.11 (IO10)
- net BUSY: now reaches U1.11 (BUSY)
- net BUSY: now also U4.5 (IO5)
- net CS1: now reaches U4.24 (RXD0)
- net CS1: now also U2.15 (~{SEL})
- net CS0: now reaches U4.25 (TXD0)
- net CS0: now also U1.5 (NSS)
- net MISO: now reaches U4.27 (IO2)
- net MISO: now also U1.2 (MISO), U2.13 (SDO)
- net CLK renamed SCK
- net SCK: now also U4.6 (IO6)
- removed net CS: U1.5 (NSS), U2.15 (~{SEL})
- net SDI renamed MOSI
- net MOSI: now also U1.3 (MOSI), U4.7 (IO7); no longer U1.2 (MISO)
- removed net SDO: U1.3 (MOSI), U2.13 (SDO)
- no-connect marks 5 -> 6

Commit message: feat(Hw):Init_BOM
Parts:
- removed C3: 1uF, Capacitor_SMD:C_0603_1608Metric, symbol Device:C_Small
- added C1: 1uF, Capacitor_SMD:C_0603_1608Metric, symbol Device:C_Small
- C12: renamed from C11; footprint (none) -> Capacitor_SMD:C_0603_1608Metric; LCSC# (none) -> C14663
- C13: renamed from C12; footprint (none) -> Capacitor_SMD:C_0603_1608Metric; LCSC# (none) -> C85713
- C14: renamed from C8; footprint (none) -> Capacitor_SMD:C_0603_1608Metric; LCSC# (none) -> C85713
- C15: renamed from C1; footprint (none) -> Capacitor_SMD:C_0603_1608Metric; LCSC# (none) -> C14663
- C16: renamed from C2; footprint (none) -> Capacitor_SMD:C_0603_1608Metric; LCSC# (none) -> C15849
- C17: renamed from C5; footprint (none) -> Capacitor_SMD:C_0603_1608Metric; LCSC# (none) -> C2241577
- C18: renamed from C7; footprint (none) -> Capacitor_SMD:C_0603_1608Metric; LCSC# (none) -> C7503509
- C19: renamed from C9; footprint (none) -> Capacitor_SMD:C_0603_1608Metric; LCSC# (none) -> C1679
- C20: renamed from C6; footprint (none) -> Capacitor_SMD:C_0603_1608Metric; LCSC# (none) -> C41361249
- C21: renamed from C10; footprint (none) -> Capacitor_SMD:C_0603_1608Metric; LCSC# (none) -> C1679
- C22: renamed from C4; footprint (none) -> Capacitor_SMD:C_0603_1608Metric; LCSC# (none) -> C519500
- L1: footprint (none) -> Inductor_SMD:L_0603_1608Metric; LCSC# C90214 -> C668512
- L2: renamed from L5; footprint (none) -> Inductor_SMD:L_0603_1608Metric; LCSC# (none) -> C86131
- L3: renamed from L2; footprint (none) -> Inductor_SMD:L_0603_1608Metric; LCSC# C701184 -> C434822
- R6: renamed from R1; footprint (none) -> Resistor_SMD:R_0603_1608Metric; LCSC# (none) -> C2930027
- renumbered AE2 to AE1, AE1 to AE2, C20 to C10, C21 to C11, C3 to C2, C13 to C3, C16 to C4, C17 to C5, C14 to C6, C15 to C7, C18 to C8, C19 to C9, R5 to R1, R8 to R2, R9 to R3, R6 to R4, R7 to R5, R3 to R7, R2 to R8, R4 to R9, SW2 to SW1, SW3 to SW2, SW1 to SW3, SW5 to SW4, SW6 to SW5, SW7 to SW6, SW4 to SW7, U4 to U1, U5 to U2, U2 to U3, U3 to U4, U1 to U5
Connections:
- net +3.3V: now also C1.1
- net GND: now also C1.2

Commit message: feat(Hw):Init_Chip_Change
Parts:
- removed U1: ESP32-C6-WROOM-1U-N4, Footprints:ESP32C6WROOM1N4, symbol Minino:ESP32-C6-WROOM-1U-N8
- added U1: ESP32-S3-WROOM-1-N8, ESP32-S3-WROOM-1_EXP, symbol Library:ESP32-S3-WROOM-1-N8
- C1: manf# TMK107BJ105KA8T -> (none)
- C10, C11, C4, C5, C8, C9: manf# KAM15AR71C104KM -> (none)
- P1: manf# TYPE-C-31-M-31 -> (none)
- R1: manf# ERJ-3GEYJ332V -> (none)
- R2, R3: manf# AC0603DR-075K1L -> (none)
- R5: manf# RMC1/16K1002DTP -> (none)
- R6: value 10K -> 100K; LCSC# C2930027 -> (none)
- R7: footprint (none) -> Resistor_SMD:R_0603_1608Metric; LCSC# (none) -> C23182
- R8, R9: footprint (none) -> Resistor_SMD:R_0603_1608Metric; LCSC# (none) -> C2907034
- SW1, SW2, SW4, SW5, SW6, SW7: manf# TL3342F160QG -> (none)
- U3: LCSC# (none) -> C476202
- U5: LCSC# (none) -> C2848401
- Y1: LCSC# (none) -> C29538
Connections:
- net +3.3V: now also U1.2 (3V3)
- net BOOT: now also U1.27 (IO0)
- net BUSY: now also U1.9 (IO16)
- net CS0: now also U1.18 (IO10)
- net CS1: now also U1.17 (IO9)
- net D+: now also U1.14 (IO20)
- net D-: now also U1.13 (IO19)
- net EN: now also U1.3 (EN)
- net GND: now also U1.1 (GND), U1.40 (GND), U1.41 (GND), U1.42 (GND), U1.43 (GND), U1.44 (GND), U1.45 (GND), U1.46 (GND), U1.47 (GND), U1.48 (GND), U1.49 (GND)
- net IRQ: now also U1.22 (IO14)
- net MISO: now also U1.21 (IO13)
- net MOSI: now also U1.19 (IO11)
- net RST: now also U1.8 (IO15)
- net SCK: now also U1.20 (IO12)
- net SCL: now also U1.10 (IO17)
- net SDA: now also U1.11 (IO18)
- net SDN: now reaches R6.2, U3.1 (SDN)
- net SDN: now also U1.12 (IO8)
- new net CS2: U1.32 (IO39)
- new net MISO2: U1.30 (IO37)
- new net MOSI2: U1.28 (IO35)
- new net SCK2: U1.29 (IO36)
Other:
- note added: "PANTALLA"
- moved on the sheet: C1, C2, C3, R1

Commit message: feat(Hw):Update_Schematic
Parts:
- removed R1: 3.3K, Resistor_SMD:R_0603_1608Metric, symbol Device:R_Small
- removed U2: XC6220B331MR-G, Package_TO_SOT_SMD:SOT-23-5, symbol HunterCat-NFC-rescue:AP2112K-3.3-Regulator_Linear
- added R3, R7, R8: 10K, Resistor_SMD:R_0603_1608Metric, symbol Device:R_Small
- added U2: BL8072CLTR33, Package_TO_SOT_SMD:SOT-223-3_TabPin2, symbol Regulator_Linear:AMS1117-3.3
- U1: footprint ESP32-S3-WROOM-1_EXP -> (none); manf# (none) -> ESP32-S3-WROOM-1-N8
- renumbered C19 to C18, C18 to C19, R2 to R1, R8 to R10, R9 to R11, R3 to R2, R7 to R9
Connections:
- net +3.3V: now also R3.2, R7.2, R8.2, U2.2 (VO); no longer R6.1
- net CS0: now also R8.1
- net CS1: now also R7.1
- net CS2: now also R3.1
- net DIO: now also U1.7 (IO7)
- net DOWN: now also U1.38 (IO2)
- net GND: now also R6.2, U2.1 (GND)
- net IO0: now also U1.23 (IO21)
- net IO1: now also U1.24 (IO47)
- net IO2: now also U1.25 (IO48)
- net IO3: now also U1.26 (IO45)
- net LEFT: now also U1.34 (IO41)
- net RIGHT: now also U1.35 (IO42)
- net SDN: now also R6.1; no longer R6.2
- net UP: now also U1.39 (IO1)
- net at C6.1, SW3.3 (A): now also U2.3 (VI)
- no-connect marks 6 -> 5
Other:
- moved on the sheet: AE2, C1, C10, C11, C12, C13, C14, C15, C16, C17, C19, C2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

Commit message: feat(Hw):Update_BOM
Parts:
- AE1: footprint (none) -> Footprints:SMA_EDGE; LCSC# (none) -> C530661
- U1: footprint (none) -> Footprints:ESP32-S3-WROOM-1_EXP
- U4: footprint (none) -> Footprints:AHT30
- Y1: footprint (none) -> Crystal:Crystal_SMD_Abracon_ABM8G-4Pin_3.2x2.5mm
Other:
- moved on the sheet: C6, C7, D1, J1, Q1, R4, SW3, U2

Commit message: feat(Hw):Update_Schematic
Parts:
- added J2: LCD, Connector_FFC-FPC:Hirose_FH12-10S-0.5SH_1x10-1MP_P0.50mm_Horizontal, symbol Connector_Generic:Conn_01x10
- AE2: LCSC# (none) -> C496553
- U5: footprint (none) -> Footprints:VGdd79S915N0S1
Connections:
- net +3.3V: now also J2.7 (Pin_7)
- net CS2: now also J2.4 (Pin_4)
- net GND: now also J2.10 (Pin_10)
- net MISO: no longer U3.13 (SDO)
- net MISO2: now also U3.13 (SDO)
- net MOSI: no longer U3.14 (SDI)
- net MOSI2: now also U3.14 (SDI)
- net SCK: no longer U3.12 (SCLK)
- net SCK2: now also U3.12 (SCLK)
- net SCL: now also J2.2 (Pin_2)
- net SDA: now also J2.1 (Pin_1)
- new net LEDA: J2.9 (Pin_9)
- new net LEDK: J2.8 (Pin_8)
- new net RS: J2.3 (Pin_3)
- new net RSTB: J2.5 (Pin_5)
- new net TE: J2.6 (Pin_6)
Other:
- moved on the sheet: C6, C7, D1, F1, J1, P1, Q1, R1, R2, R4, R6, SW3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

Commit message: feat(Hw):Update_Schematic
Parts:
- removed AE2: Antenna_Shield, symbol Device:Antenna_Shield
- added AE2: Antenna, Connector_PinHeader_2.54mm:PinHeader_1x01_P2.54mm_Vertical, symbol Device:Antenna
- added R12: 47r, Resistor_SMD:R_0603_1608Metric, symbol Device:R
- J2: LCSC# C2856816 -> C2856816 o C262583
- R6: LCSC# (none) -> C25803
Connections:
- net LEDK is gone; now on net GND: J2.8 (Pin_8)
- net +3.3V: now also R12.1
- net BUSY: now also U1.16 (IO46); no longer U1.9 (IO16)
- net CS0: now also U1.8 (IO15); no longer U1.18 (IO10)
- net CS1: now also J2.4 (Pin_4), R3.1, U1.18 (IO10); no longer R7.1, U1.17 (IO9), U3.15 (~{SEL})
- net CS2: now also R7.1, U1.31 (IO38), U3.15 (~{SEL}); no longer J2.4 (Pin_4), R3.1, U1.32 (IO39)
- net DIO: now also U1.4 (IO4); no longer U1.7 (IO7)
- net DOWN: now also U1.23 (IO21); no longer U1.38 (IO2)
- net IO0: now also U1.25 (IO48); no longer U1.23 (IO21)
- net IO1: now also U1.26 (IO45); no longer U1.24 (IO47)
- net IO2: now also U1.34 (IO41); no longer U1.25 (IO48)
- net IO3: now also U1.35 (IO42); no longer U1.26 (IO45)
- net IRQ: now also U1.32 (IO39); no longer U1.22 (IO14)
- net LEDA: now also R12.2
- net LEFT: now also U1.21 (IO13); no longer U1.34 (IO41)
- net MISO: now also U1.10 (IO17); no longer U1.21 (IO13)
- net MISO2: now also U1.29 (IO36); no longer U1.30 (IO37)
- net MOSI: now also U1.9 (IO16); no longer U1.19 (IO11)
- net RIGHT: now also U1.22 (IO14); no longer U1.35 (IO42)
- net RS: now also U1.17 (IO9)
- net RST: now also U1.15 (IO3); no longer U1.8 (IO15)
- net RSTB: now also U1.12 (IO8)
- net SCK: now also U1.11 (IO18); no longer U1.20 (IO12)
- net SCK2: now also U1.30 (IO37); no longer U1.29 (IO36)
- net SCL: now also U1.20 (IO12); no longer R10.2, U1.10 (IO17), U4.3 (SCL)
- net SDA: now also U1.19 (IO11); no longer R11.2, U1.11 (IO18), U4.4 (SDA)
- net SDN: now also U1.33 (IO40); no longer U1.12 (IO8)
- net TE: now also U1.7 (IO7)
- net UP: now also U1.24 (IO47); no longer U1.39 (IO1)
- net at C22.2: now also AE2.1 (A)
- net SDA1: now reaches U1.5 (IO5)
- net SDA1: now also R11.2, U4.4 (SDA)
- net SCL1: now reaches U1.6 (IO6)
- net SCL1: now also R10.2, U4.3 (SCL)
Other:
- moved on the sheet: J2, R3
