File: hardware/Badge_Tropicon_2026.kicad_sch (KiCad schematic)
At the start: 63 parts, among them J1 Battery, J2 LCD, P1 USB_C_Plug_USB2.0, Q1 DMG3415U-7, Q2 BC846, SW3 ON, U1 ESP32-S3-WROOM-1-N8, U2 BL8072CLTR33, U3 Si4463, U4 AHT30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

Commit message: feat(Hw):3D_Model_Added
Other:
- company: (none) -> Electronic Cats
- title: (none) -> Badge Tropicon 2026
Changed lines of the file:
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@@
 	(generator_version "9.0")
 	(paper "A3")
+	(title_block
+		(title "Badge Tropicon 2026")
+		(date "2026-02-27")
+		(rev "v1.0")
+		(company "Electronic Cats")
+		(comment 1 "Lizeth Gallegos Martínez")
+	)
 	(text "REGULATOR"
 		(exclude_from_sim no)

Commit message: feat(Hw):Update_BOM
Parts:
- R16: LCSC# (none) -> C2906974
Changed lines of the file:
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@@
 			)
 		)
-		(property "LCSC#" ""
+		(property "LCSC#" "C2906974"
 			(at 379.73 162.56 90)
 			(effects
