File: hardware/Badge_Tropicon_2026.kicad_pcb (KiCad board)
At the start: 2 copper layers, 99.7 x 100 mm, 64 parts, among them J1 Battery, J2 LCD, P1 USB_C_Plug_USB2.0, Q1 DMG3415U-7, Q2 BC846, SW3 ON, U1 ESP32-S3-WROOM-1-N8, U2 BL8072CLTR33, U3 Si4463, U4 AHT30, U5 VGdd79S915N0S1, Y1 30MHz

Commit message: feat(Hw):3D_Model_Added
Changed lines of the file:
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@@
 	)
 	(paper "A4")
+	(title_block
+		(title "Badge Tropicon 2026")
+		(date "2026-02-27")
+		(rev "v1.0")
+		(company "Electronic Cats")
+		(comment 1 "Lizeth Gallegos Martínez")
+	)
 	(layers
 		(0 "F.Cu" signal)
@@
 		)
 		(embedded_fonts no)
+		(model "${KIPRJMOD}/Footprints/3D/ER-TFT2.79-1.step"
+			(offset
+				(xyz 0 0 0)
+			)
+			(scale
+				(xyz 1 1 1)
+			)
+			(rotate
+				(xyz 0 0 0)
+			)
+		)
 	)
 	(footprint "Capacitor_SMD:C_0603_1608Metric"
@@
 	)
 	(segment
+		(start 116.16 97.09237)
+		(end 115.947066 96.879436)
+		(width 0.2)
+		(layer "B.Cu")
+		(net 32)
+	)
+	(segment
 		(start 182.675167 89.35)
 		(end 182.685167 89.34)
@@
 	)
 	(segment
-		(start 115.947066 102.117066)
-		(end 115.947066 96.879436)
+		(start 116.16 102.33)
+		(end 116.16 97.09237)
 		(width 0.2)
 		(layer "B.Cu")
@@
 	(segment
 		(start 116.645 102.815)
-		(end 115.947066 102.117066)
+		(end 116.16 102.33)
 		(width 0.2)
 		(layer "B.Cu")
@@
 	)
 	(segment
-		(start 115.759 103.649)
-		(end 181.371 103.649)
+		(start 181.371 103.649)
+		(end 182.93 102.09)
 		(width 0.2)
 		(layer "F.Cu")
@@
 	)
 	(segment
-		(start 184.11 92.38)
-		(end 188.96 92.38)
+		(start 115.759 103.649)
+		(end 181.371 103.649)
 		(width 0.2)
 		(layer "F.Cu")
@@
 	)
 	(segment
-		(start 190.05 91.29)
-		(end 190.05 89.46)
+		(start 182.93 102.09)
+		(end 182.93 93.56)
 		(width 0.2)
 		(layer "F.Cu")
@@
 	)
 	(segment
-		(start 115.185 103.075)
-		(end 115.759 103.649)
+		(start 182.93 93.56)
+		(end 184.11 92.38)
 		(width 0.2)
 		(layer "F.Cu")
@@
 	)
 	(segment
-		(start 181.371 103.649)
-		(end 182.93 102.09)
+		(start 190.05 91.29)
+		(end 190.05 89.46)
 		(width 0.2)
 		(layer "F.Cu")
@@
 	)
 	(segment
-		(start 182.93 102.09)
-		(end 182.93 93.56)
+		(start 115.005 102.895)
+		(end 115.759 103.649)
 		(width 0.2)
 		(layer "F.Cu")
@@
 	)
 	(segment
-		(start 182.93 93.56)
-		(end 184.11 92.38)
+		(start 188.96 92.38)
+		(end 190.05 91.29)
 		(width 0.2)
 		(layer "F.Cu")
@@
 	)
 	(segment
-		(start 188.96 92.38)
-		(end 190.05 91.29)
+		(start 184.11 92.38)
+		(end 188.96 92.38)
 		(width 0.2)
 		(layer "F.Cu")
@@
 	)
 	(via
-		(at 115.185 103.075)
+		(at 115.005 102.895)
 		(size 0.6)
 		(drill 0.3)
@@
 	)
 	(segment
-		(start 114.703903 102.593903)
-		(end 114.703903 97.139149)
-		(width 0.2)
-		(layer "B.Cu")
-		(net 38)
-	)
-	(segment
 		(start 190.05 84.38)
 		(end 191.09 83.34)
@@
 	)
 	(segment
-		(start 115.185 103.075)
+		(start 114.703903 102.593903)
+		(end 114.703903 97.139149)
+		(width 0.2)
+		(layer "B.Cu")
+		(net 38)
+	)
+	(segment
+		(start 115.005 102.895)
 		(end 114.703903 102.593903)
 		(width 0.2)

Commit message: feat(Hw):Update_Route
Parts:
- moved C20 2.11 mm to (146.9, 87.8)
- moved U3 2.11 mm to (146.4, 93.9)
- moved C19 2.11 mm to (150.0, 92.1)
- moved L1 2.11 mm to (146.1, 90.0)
- moved R7 2.11 mm to (144.6, 98.2)
- moved C16 2.11 mm to (152.9, 92.1)
- moved Y1 2.11 mm to (141.4, 94.8)
- moved C15 2.11 mm to (151.4, 92.1)
- moved R6 1.64 mm to (142.0, 91.7)
- moved L3 1.11 mm to (145.4, 87.8), turned to 90 degrees
- moved SW3 0.09 mm to (111.5, 146.6)
Routing:
- net GND: track 28.7 -> 47.7 mm, vias 121 -> 124
- net /IRQ: track 35.7 -> 38.6 mm
- net /MOSI2: track 35.8 -> 38.6 mm
- net /MISO2: track 36.1 -> 38.9 mm
- net /CS2: track 29.5 -> 32.0 mm
- net +3.3V: track 336.1 -> 338.1 mm
- net /Rxp: track 6.64 -> 5.00 mm
- net /IO0: track 43.9 -> 45.1 mm
- net /IO1: track 38.3 -> 39.0 mm
Other:
- board text removed: "${REFERENCE}"
