File: hardware/Badge_Tropicon_2026.kicad_pcb (KiCad board)
At the start: 2 copper layers, 99.7 x 100 mm, 64 parts, among them J1 Battery, J2 LCD, P1 USB_C_Plug_USB2.0, Q1 DMG3415U-7, Q2 BC846, SW3 ON, U1 ESP32-S3-WROOM-1-N8, U2 BL8072CLTR33, U3 Si4463, U4 AHT30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

Commit message: feat(Hw):Uppdate_Route
Routing:
- net /MISO: track 94.5 -> 92.3 mm
- net /IO1: track 39.0 -> 38.4 mm
- net /MOSI: track 90.6 -> 91.1 mm
