File: hardware/Add-On/Addon-Cerveza/Addon-Cerveza.kicad_sch (KiCad schematic)
At the start: 12 parts, among them J1 Conn_02x03_Odd_Even, SW2 On, SW7 RESET, U1 TMP102xxDRL, U2 CH32V003F4U6

Commit message: feat(Hw):Init_Floorplan_Add-On_Cerveza
Parts:
- added R1, R2, R3: 5K, Resistor_SMD:R_0603_1608Metric, symbol Device:R
- BT1: footprint Library:BAT-HLD-001 -> Footprints:BAT-HLD-001
- C16, R6: provedor LCSC -> (none)
- D11: footprint LED_SMD:LED_WS2812B-Mini_PLCC4_3.5x3.5mm -> Footprints:LED_SK6812-E; LCSC# C527089 -> C5378731; provedor LCSC -> (none)
- J1: footprint Library:B-2100N06P-B111_CKM -> Footprints:B-2100N06P-B111_CKM
- SW2: footprint Library:MSK12C02 -> Footprints:MSK12C02
Connections:
- net USB_DET is gone; now on net SCL: U2.12 (PC2)
- net +3V3: now also R1.1, R2.1, R3.1
- net SDA: now reaches U2.11 (PC1)
- net SDA: now also U1.6 (SDA), R1.2
- net ALERT: now reaches U2.8 (PD0)
- net ALERT: now also U1.3 (ALERT), R3.2
- net SCL: now reaches U1.1 (SCL)
- net SCL: now also R2.2
- net BTN_1: no longer names the net of U2.3 (PD6)
- net BTN_2: no longer names the net of U2.2 (PD5)
- net D+: no longer names the net of U2.20 (PD3)
- net D-: no longer names the net of U2.19 (PD2)
- no-connect marks 12 -> 15
Other:
- company: (none) -> Electronic Cats
- title: (none) -> Addon-Cerveza
- moved on the sheet: C1, U1

Commit message: feat(Hw):Update_Schematic_And_Route_Addon_Cerveza
Parts:
- added JP1: Jumper, Jumper:SolderJumper-2_P1.3mm_Bridged_RoundedPad1.0x1.5mm, symbol Jumper:Jumper_2_Bridged
- added R4: 10k, Resistor_SMD:R_0603_1608Metric, symbol Device:R
- R1, R2: value 5K -> 4.7K; LCSC# C3202451 -> C2907034
- R3: value 5K -> 10k; LCSC# C3202451 -> C2930027
Connections:
- net GND: now also JP1.1 (A); no longer U1.4 (ADD0)
- new net: JP1.2 (B), R4.1
- new net: R4.2, U1.4 (ADD0)
Other:
- moved on the sheet: C1, R1, R2, R3, U1
