File: hardware/Add-On/Addon-Websec/Addon-Websec.kicad_pcb (KiCad board)
At the start: 2 copper layers, 45.6 x 50 mm, 22 parts, among them J3 Conn_02x03_Odd_Even, SW5 SW_RST, SW6 On, U3 PY32F002AA15M6TU

Commit message: feat(Hw):Update_Route_Websec
Connections:
- D13 pad 2: /PA6 -> /PA1
- D14 pad 2: /PA7 -> /PA6
Routing:
- net /PA1: track 0.00 -> 23.0 mm, vias 0 -> 1
- net /PA7: track 16.6 -> 0.00 mm, vias 1 -> 0
- net /PA6: track 18.1 -> 15.8 mm, vias 1 -> 3
- net /PF0: track 22.3 -> 22.1 mm, vias 1 -> 3
- net /SWCLK: track 27.0 -> 27.1 mm, vias 0 -> 2
- net /GND: vias 6 -> 13
