File: hardware/Add-On/Addon-Websec/Addon-Websec.kicad_sch (KiCad schematic)
At the start: 14 parts, among them J3 Conn_02x03_Odd_Even, SW5 SW_RST, SW6 On, U3 PY32F002AA15M6TU

Commit message: feat(Hw):Update_Schematic_And_Route_Addon_Cerveza
Other:
- company: (none) -> Electronic Cats
- title: (none) -> Addon-Websec
Changed lines of the file:
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@@
 	(generator_version "9.0")
 	(paper "A5")
+	(title_block
+		(title "Addon-Websec")
+		(date "2026-03-09")
+		(rev "v1.0")
+		(company "Electronic Cats")
+		(comment 1 "Lizeth Gallegos Martínez")
+	)
 	(text "Battery"
 		(exclude_from_sim no)

Commit message: feat(Hw):Update_Route_Websec
Connections:
- net PA1: now also D13.2 (A)
- net PA6: now also D14.2 (A); no longer D13.2 (A)
- net PA7: no longer D14.2 (A)
Changed lines of the file:
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@@
 	(wire
 		(pts
-			(xy 191.135 69.85) (xy 187.96 69.85)
+			(xy 191.77 69.85) (xy 187.96 69.85)
 		)
 		(stroke
@@
 	(wire
 		(pts
-			(xy 191.135 66.04) (xy 191.135 69.85)
+			(xy 191.77 66.04) (xy 191.77 69.85)
 		)
 		(stroke
@@
 		)
 	)
+	(label "PA1"
+		(at 191.77 66.04 0)
+		(effects
+			(font
+				(size 1.27 1.27)
+			)
+			(justify left bottom)
+		)
+	)
 	(label "PA6"
-		(at 191.135 66.04 0)
+		(at 190.5 81.28 0)
 		(effects
 			(font
@@
 		)
 	)
-	(label "PA7"
-		(at 190.5 81.28 0)
-		(effects
-			(font
-				(size 1.27 1.27)
-			)
-			(justify left bottom)
-		)
-	)
